File: _autosave-weather_external.sch (KiCad schematic (older format))
At the start: 20 parts, among them J2 22-23-2021, J3 640456-3, J4 22-23-2021, J5 Conn_02x04_Odd_Even, SW1 SW_Push, U1 ATMEGA328-PU, U2 NE555DR, U5 DHT11, Y1 Crystal

Commit message: Print version 1
Parts:
- added C7: C, Capacitor_THT:C_Disc_D3.0mm_W1.6mm_P2.50mm, symbol Device:C
- C6: renamed from C?; footprint (none) -> Capacitor_THT:C_Disc_D3.0mm_W1.6mm_P2.50mm
Connections:
- net GND: now also C7.2
- net at U1.13 (PD7), U5.1 (VCC): now also C7.1
Changed lines of the file:
@@
 $EndComp
-Wire Wire Line
-	6050 6150 5150 6150
 Wire Wire Line
 	5150 6750 5600 6750
@@
 	4250 6050 6500 6050
 $Comp
-L Device:C C?
+L Device:C C6
 U 1 1 5F852F52
 P 2600 6050
-F 0 "C?" V 2852 6050 50  0000 C CNN
+F 0 "C6" V 2852 6050 50  0000 C CNN
 F 1 "C" V 2761 6050 50  0000 C CNN
-F 2 "" H 2638 5900 50  0001 C CNN
+F 2 "Capacitor_THT:C_Disc_D3.0mm_W1.6mm_P2.50mm" H 2638 5900 50  0001 C CNN
 F 3 "~" H 2600 6050 50  0001 C CNN
 	1    2600 6050
@@
 Wire Wire Line
 	2350 6400 2500 6400
+$Comp
+L Device:C C7
+U 1 1 5F877CE5
+P 4250 6450
+F 0 "C7" H 4365 6496 50  0000 L CNN
+F 1 "C" H 4365 6405 50  0000 L CNN
+F 2 "Capacitor_THT:C_Disc_D3.0mm_W1.6mm_P2.50mm" H 4288 6300 50  0001 C CNN
+F 3 "~" H 4250 6450 50  0001 C CNN
+	1    4250 6450
+	1    0    0    -1
+$EndComp
+Wire Wire Line
+	4250 6150 4250 6300
+Wire Wire Line
+	4250 6150 5150 6150
+Connection ~ 5150 6150
+Wire Wire Line
+	5150 6150 6050 6150
+Wire Wire Line
+	4250 6600 4250 6750
+Wire Wire Line
+	4250 6750 5150 6750
+Connection ~ 5150 6750
 $EndSCHEMATC
