File: weather_external.kicad_pcb (KiCad board)
At the start: 2 copper layers, 38 x 56.4 mm, 20 parts, among them J2 22-23-2021, J3 640456-3, J4 22-23-2021, SW1 SW_Push, U4 MCP1700-3302E_SOT23

Commit message: Print version 1
Parts:
- removed Atmega328: ATMEGA328-PU, digikey-footprints:DIP-28_W7.62mm
- removed U4: MCP1700-3302E_SOT23, Package_TO_SOT_SMD:SOT-23
- added C6: C, Capacitor_THT:C_Disc_D3.0mm_W1.6mm_P2.50mm, F.Cu at (141.7, 116.9)
- added C7: C, Capacitor_THT:C_Disc_D3.0mm_W1.6mm_P2.50mm, F.Cu at (134.7, 110.6)
- added U1: ATMEGA328-PU, digikey-footprints:DIP-28_W7.62mm, F.Cu at (144.8, 73.7)
- moved D1 31.1 mm to (134.1, 88.2)
- moved C5 26.4 mm to (135.8, 58.1)
- moved J5 24.4 mm to (144.9, 116.9), turned to 90 degrees
- moved R2 22.3 mm to (142.4, 85.6), turned to 180 degrees
- moved U5 15.1 mm to (139.8, 106.4), turned to 270 degrees
- moved J2 12.8 mm to (140.8, 88.8), turned to 270 degrees
- moved R1 12.0 mm to (131.0, 85.0)
- moved C2 9.94 mm to (136.2, 98.7)
- moved C1 9.94 mm to (133.4, 96.2)
- moved SW1 5.34 mm to (127.1, 63.4)
- moved R3 3.83 mm to (140.3, 57.7)
- moved R4 2.50 mm to (144.5, 57.7)
- moved C4 2.06 mm to (142.5, 81.8)
- moved U2 2.01 mm to (148.4, 65.6)
- moved J3 1.81 mm to (141.0, 78.4)
- renumbered NRF24l01 to J5, 555 to U2, DHT11 to U5, 16MHz to Y1
Connections:
- J5 pad 2: Net-(J5-Pad2) -> VCC
Routing:
- net VCC: track 84.4 -> 187.1 mm
- net Net-(J5-Pad5): track 10.7 -> 42.7 mm
- net Net-(J5-Pad2): track 23.2 -> 0.00 mm
- net Net-(C4-Pad1): track 27.0 -> 47.9 mm
- net Net-(J5-Pad7): track 13.4 -> 29.8 mm
- net Net-(J5-Pad6): track 10.3 -> 22.7 mm
- net Net-(R2-Pad1): track 12.8 -> 3.12 mm
- net Net-(C5-Pad1): track 26.6 -> 31.7 mm
- net Net-(J5-Pad3): track 23.4 -> 27.3 mm
- net Net-(C1-Pad1): track 16.3 -> 13.2 mm
- net Net-(J5-Pad4): track 10.8 -> 13.5 mm
- net Net-(C7-Pad1): track 15.8 -> 13.2 mm
- net Net-(R3-Pad1): track 17.2 -> 19.7 mm
- net Net-(J3-Pad1): track 6.12 -> 3.92 mm
- net Net-(D1-Pad1): track 4.68 -> 2.68 mm
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- removed copper zone on B.Cu, net GND
Other:
- board outline removed
- board text added: "Weather Ext PV1.0"
- board text removed: "Led on/off"
