File: weather_external.kicad_pcb (KiCad board)
At the start: 2 copper layers, 38 x 56.4 mm, 20 parts, among them J2 22-23-2021, J3 640456-3, J4 22-23-2021, SW1 SW_Push, U4 MCP1700-3302E_SOT23

Commit message: Weather External v1.0
Parts:
- added C6: C, Capacitor_THT:C_Disc_D3.0mm_W1.6mm_P2.50mm, F.Cu at (164.8, 107.8)
- added C7: C, Capacitor_THT:C_Disc_D3.0mm_W1.6mm_P2.50mm, F.Cu at (135.1, 98.5)
- added JP1: Jumper, SolderJumper:SolderJumper-2_P1.3mm_Open_Pad1.0x1.5mm, F.Cu at (161.9, 79.5)
- renumbered 16MHz to 16Mhz, 555 to NE555, NRF24l01 to NRF24L01
Connections:
- Atmega328 pad 11: Net-(R2-Pad1) -> (no net)
- Atmega328 pad 13: (no net) -> Net-(C7-Pad2)
- Atmega328 pad 5: (no net) -> Net-(R2-Pad1)
- Atmega328 pad 6: Net-(U1-Pad6) -> (no net)
- DHT11 pad 1: Net-(U1-Pad12) -> Net-(C7-Pad2)
- DHT11 pad 2: Net-(U1-Pad6) -> Net-(U1-Pad12)
Routing:
- net Net-(C7-Pad2): track 0.00 -> 21.4 mm
- net Net-(C6-Pad1): track 23.2 -> 36.4 mm
- net Net-(R2-Pad1): track 12.8 -> 25.0 mm
- net Net-(U1-Pad6): track 11.9 -> 0.00 mm
- net Net-(U1-Pad12): track 15.8 -> 19.0 mm
- net VCC: track 84.4 -> 87.5 mm
- net Net-(J5-Pad7): track 13.4 -> 12.8 mm
